Commit message: update model

File: ROS2/dual_piper_v2/urdf/brainco-lefthand-URDF-V2.urdf (robot description, URDF)
Before this commit: robot brainco-lefthand-URDF-V2, 17 links, 16 joints
Links:
- removed link left_base_link
- removed link left_index_distal_Link
- removed link left_index_proximal_Link
- removed link left_index_tip_Link
- removed link left_middle_distal_Link
- removed link left_middle_proximal_Link
- removed link left_middle_tip_Link
- removed link left_pinky_distal_Link
- removed link left_pinky_proximal_Link
- removed link left_pinky_tip_Link
- removed link left_ring_distal_Link
- removed link left_ring_proximal_Link
- removed link left_ring_tip_Link
- removed link left_thumb_distal_Link
- removed link left_thumb_metacarpal_Link
- removed link left_thumb_proximal_Link
- removed link left_thumb_tip_Link
Joints:
- removed joint left_index_distal_joint
- removed joint left_index_proximal_joint
- removed joint left_index_tip_joint
- removed joint left_middle_distal_joint
- removed joint left_middle_proximal_joint
- removed joint left_middle_tip_joint
- removed joint left_pinky_distal_joint
- removed joint left_pinky_proximal_joint
- removed joint left_pinky_tip_joint
- removed joint left_ring_distal_joint
- removed joint left_ring_proximal_joint
- removed joint left_ring_tip_joint
- removed joint left_thumb_distal_joint
- removed joint left_thumb_metacarpal_joint
- removed joint left_thumb_proximal_joint
- removed joint left_thumb_tip_joint

File: ROS2/dual_piper_v2/urdf/brainco-righthand-URDF-V2.urdf (robot description, URDF)
Before this commit: robot brainco-righthand-URDF-V2, 17 links, 16 joints
Links:
- removed link right_base_link
- removed link right_index_distal_link
- removed link right_index_proximal_link
- removed link right_index_tip
- removed link right_middle_distal_link
- removed link right_middle_proximal_link
- removed link right_middle_tip
- removed link right_pinky_distal_link
- removed link right_pinky_proximal_link
- removed link right_pinky_tip
- removed link right_ring_distal_link
- removed link right_ring_proximal_link
- removed link right_ring_tip
- removed link right_thumb_distal_link
- removed link right_thumb_metacarpal_link
- removed link right_thumb_proximal_link
- removed link right_thumb_tip
Joints:
- removed joint right_index_distal_joint
- removed joint right_index_proximal_joint
- removed joint right_index_tip_joint
- removed joint right_middle_distal_joint
- removed joint right_middle_proximal_joint
- removed joint right_middle_tip_joint
- removed joint right_pinky_distal_joint
- removed joint right_pinky_proximal_joint
- removed joint right_pinky_tip_joint
- removed joint right_ring_distal_joint
- removed joint right_ring_proximal_joint
- removed joint right_ring_tip_joint
- removed joint right_thumb_distal_joint
- removed joint right_thumb_metacarpal_joint
- removed joint right_thumb_proximal_joint
- removed joint right_thumb_tip

File: ROS2/dual_piper_v2/urdf/piper_description_with_camera_front_left.xacro (robot description, xacro)
@@ -2,4 +2,7 @@
 <robot xmlns:xacro="http://www.ros.org/wiki/xacro" name="piper_camera">
     <xacro:macro name="front_left" params="namespace">
+    <xacro:include filename="$(find dual_piper_v2)/urdf/brainco-lefthand-URDF-V2.urdf"/>
+    <xacro:left namespace="${namespace}">
+    </xacro:left>
     <link name="${namespace}/arm_base">
         <inertial>
@@ -254,5 +257,12 @@
         <limit lower="-3.14" upper="3.14" effort="100" velocity="3" />
     </joint>
-    <link name="${namespace}/link7">
+    <joint name="${namespace}/hand_joint" type="fixed">
+        <origin xyz="0.00 0.0 0.065" rpy="0.0 0.0 -1.57"/>
+        <parent link="${namespace}/link6"/>
+        <child link="${namespace}/left_base_link"/>
+        <axis xyz="0.0 0.0 0.0"/>
+        <limit lower="0.0" upper="0.0" effort="0.0" velocity="0.0"/>
+    </joint>
+    <!-- <link name="${namespace}/link7">
         <inertial>
         <origin
@@ -327,5 +337,5 @@
         <axis xyz="0 0 1" />
         <limit lower="-0.05" upper="0" effort="100" velocity="1" />
-    </joint>
+    </joint> -->
 </xacro:macro>
 </robot>

File: ROS2/dual_piper_v2/urdf/piper_hand.xacro (robot description, xacro)
@@ -1,9 +1,7 @@
 <?xml version="1.0"?>
-<robot xmlns:xacro="http://www.ros.org/wiki/xacro" name="piper_camera">
-    <xacro:macro name="front_right" params="namespace">
-    <xacro:include filename="$(find dual_piper_v2)/urdf/brainco-righthand-URDF-V2.urdf"/>
-    <xacro:left namespace="${namespace}">
-    </xacro:left>
-    <link name="${namespace}/arm_base">
+<robot xmlns:xacro="http://www.ros.org/wiki/xacro" name="piper_fl">
+    <xacro:macro name="namespace" params="namespace">
+    <xacro:include filename="$(find dual_piper_v2)/urdf/brainco-lefthand-URDF-V2.urdf"/>
+   <link name="${namespace}/arm_base">
         <inertial>
         <origin
@@ -22,5 +20,5 @@
         <origin xyz="0 0 0" rpy="0 0 0" />
         <geometry>
-            <mesh filename="package://dual_piper_v2/meshes/dae/base_link.dae" />
+            <mesh filename="package://dual_piper_v2/meshes/base_link.dae" />
         </geometry>
         <material name="">
@@ -31,5 +29,5 @@
             <origin xyz="0 0 0" rpy="0 0 0" />
             <geometry>
-                <mesh filename="package://dual_piper_v2/meshes/base_link.STL" />
+                <mesh filename="package://dual_piper_v2/meshes/base_link.dae" />
             </geometry>
         </collision>
@@ -52,12 +50,12 @@
         <origin xyz="0 0 0" rpy="0 0 0" />
         <geometry>
-            <mesh filename="package://dual_piper_v2/meshes/dae/link1.dae" />
-        </geometry>
-        <material name="">
-            <color rgba="0.792156862745098 0.819607843137255 0.933333333333333 1" />
-        </material>
-        </visual>
-        <collision>
-            <origin xyz="0 0 0" rpy="0 0 1.5708" />
+            <mesh filename="package://dual_piper_v2/meshes/link1.dae" />
+        </geometry>
+        <material name="">
+            <color rgba="0.792156862745098 0.819607843137255 0.933333333333333 1" />
+        </material>
+        </visual>
+        <collision>
+            <origin xyz="0 0 0" rpy="0 0 0" />
             <geometry>
                 <mesh filename="package://dual_piper_v2/meshes/link1.STL" />
@@ -89,12 +87,12 @@
         <origin xyz="0 0 0" rpy="0 0 0" />
         <geometry>
-            <mesh filename="package://dual_piper_v2/meshes/dae/link2.dae" />
-        </geometry>
-        <material name="">
-            <color rgba="0.792156862745098 0.819607843137255 0.933333333333333 1" />
-        </material>
-        </visual>
-        <collision>
-            <origin xyz="0 0 0" rpy="0 0 0.1" />
+            <mesh filename="package://dual_piper_v2/meshes/link2.dae" />
+        </geometry>
+        <material name="">
+            <color rgba="0.792156862745098 0.819607843137255 0.933333333333333 1" />
+        </material>
+        </visual>
+        <collision>
+            <origin xyz="0 0 0" rpy="0 0 0" />
             <geometry>
                 <mesh filename="package://dual_piper_v2/meshes/link2.STL" />
@@ -103,5 +101,5 @@
     </link>
     <joint name="${namespace}/joint2" type="revolute">
-        <origin xyz="0 0 0" rpy="1.5708 -0.034907 -1.5708" />
+        <origin xyz="0 0 0" rpy="1.5708 0 -1.5708" />
         <parent link="${namespace}/link1" />
         <child link="${namespace}/link2" />
@@ -126,12 +124,12 @@
         <origin xyz="0 0 0" rpy="0 0 0" />
         <geometry>
-            <mesh filename="package://dual_piper_v2/meshes/dae/link3.dae" />
-        </geometry>
-        <material name="">
-            <color rgba="0.792156862745098 0.819607843137255 0.933333333333333 1" />
-        </material>
-        </visual>
-        <collision>
-        <origin xyz="0 0 0" rpy="0 0 -1.75" />
+            <mesh filename="package://dual_piper_v2/meshes/link3.dae" />
+        </geometry>
+        <material name="">
+            <color rgba="0.792156862745098 0.819607843137255 0.933333333333333 1" />
+        </material>
+        </visual>
+        <collision>
+        <origin xyz="0 0 0" rpy="0 0 0" />
         <geometry>
             <mesh filename="package://dual_piper_v2/meshes/link3.STL" />
@@ -140,5 +138,5 @@
     </link>
     <joint name="${namespace}/joint3" type="revolute">
-        <origin xyz="0.28358 0.028726 0" rpy="0 0 0.06604341" />
+        <origin xyz="0.28358 0.028726 0" rpy="0 0 0.10095" />
         <parent link="${namespace}/link2" />
         <child link="${namespace}/link3" />
@@ -163,5 +161,5 @@
         <origin xyz="0 0 0" rpy="0 0 0" />
         <geometry>
-            <mesh filename="package://dual_piper_v2/meshes/dae/link4.dae" />
+            <mesh filename="package://dual_piper_v2/meshes/link4.dae" />
         </geometry>
         <material name="">
@@ -200,12 +198,12 @@
         <origin xyz="0 0 0" rpy="0 0 0" />
         <geometry>
-            <mesh filename="package://dual_piper_v2/meshes/dae/link5.dae" />
-        </geometry>
-        <material name="">
-            <color rgba="0.792156862745098 0.819607843137255 0.933333333333333 1" />
-        </material>
-        </visual>
-        <collision>
-        <origin xyz="0 0 0" rpy="0 0 -3.14" />
+            <mesh filename="package://dual_piper_v2/meshes/link5.dae" />
+        </geometry>
+        <material name="">
+            <color rgba="0.792156862745098 0.819607843137255 0.933333333333333 1" />
+        </material>
+        </visual>
+        <collision>
+        <origin xyz="0 0 0" rpy="0 0 0" />
         <geometry>
             <mesh filename="package://dual_piper_v2/meshes/link5.STL" />
@@ -235,16 +233,16 @@
         </inertial>
         <visual>
-        <origin xyz="-0.002 -0.008 0" rpy="-1.57 0 0" />
-        <geometry>
-            <mesh filename="package://dual_piper_v2/meshes/dae/camera_v3.dae"/>
-        </geometry>
-        <material name="">
-            <color rgba="0.792156862745098 0.819607843137255 0.933333333333333 1" />
-        </material>
-        </visual>
-        <collision>
-        <origin xyz="-0.002 -0.008 0" rpy="-1.57 0 0" />
-        <geometry>
-            <mesh filename="package://dual_piper_v2/meshes/dae/camera_v3.dae"/>
+        <origin xyz="0 0 0" rpy="0 0 0" />
+        <geometry>
+            <mesh filename="package://dual_piper_v2/meshes/link6.STL" />
+        </geometry>
+        <material name="">
+            <color rgba="0.792156862745098 0.819607843137255 0.933333333333333 1" />
+        </material>
+        </visual>
+        <collision>
+        <origin xyz="0 0 0" rpy="0 0 0" />
+        <geometry>
+            <mesh filename="package://dual_piper_v2/meshes/link6.STL" />
         </geometry>
         </collision>
@@ -257,85 +255,40 @@
         <limit lower="-3.14" upper="3.14" effort="100" velocity="3" />
     </joint>
-    <joint name="${namespace}/hand_joint" type="fixed">
-        <origin xyz="0.00 0.0 0.065" rpy="0.0 0.0 -1.57"/>
+    <!-- <link name="${namespace}/lidar_end_link">
+        <inertial>
+            <origin xyz="0.0 0.0 0.0" rpy="0.0 0.0 0.0"/>
+            <mass value="2.0"/>
+            <inertia ixx="0.0" ixy="0.0" ixz="0.0" iyy="0.0" iyz="0.0" izz="0.0"/>
+        </inertial>
+        <visual name="">
+            <origin xyz="0.0 0.0 0.0" rpy="0.0 3.14 0.0"/>
+            <geometry>
+                <mesh filename="package://dual_piper_v2/meshes/dae/lidar_end_v2.stl" scale="0.1 0.1 0.1"/>
+            </geometry>
+            <material name="">
+                <color rgba="1.0 0.0 0.0 1.0"/>
+                <texture filename=""/>
+            </material>
+        </visual>
+        <collision>
+            <origin xyz="0.0 0.0 0.0" rpy="0.0 3.14 0.0"/>
+            <geometry>
+                <mesh filename="package://dual_piper_v2/meshes/dae/lidar_end_v2.stl" scale="0.1 0.1 0.1"/>
+            </geometry>
+        </collision>
+    </link>
+    <joint name="${namespace}/lidar_end_joint" type="fixed">
+        <origin xyz="0.00 0.018 0.09" rpy="0.0 0.0 0.0"/>
         <parent link="${namespace}/link6"/>
-        <child link="${namespace}/right_base_link"/>
+        <child link="${namespace}/lidar_end_link"/>
+        <axis xyz="0.0 0.0 0.0"/>
+    </joint> -->
+    <joint name="hand_joint" type="fixed">
+        <origin xyz="0.0 0.0 0.0" rpy="0.0 0.0 0.0"/>
+        <parent link="${namespace}/link6"/>
+        <child link="${namespace}/left_base_link"/>
         <axis xyz="0.0 0.0 0.0"/>
         <limit lower="0.0" upper="0.0" effort="0.0" velocity="0.0"/>
     </joint>
-    <!-- <link name="${namespace}/link7">
-        <inertial>
-        <origin
-            xyz="-0.000277778383727112 -0.0467673043650824 -0.00921029491873201"
-            rpy="0 0 0" />
-        <mass value="0.02648229234527" />
-        <inertia
-            ixx="9.99787479924589E-06"
-            ixy="-1.57548495096104E-07"
-            ixz="-2.71342775003487E-08"
-            iyy="6.1795212293655E-06"
-            iyz="-1.58939803580081E-06"
-            izz="1.42102717246564E-05" />
-        </inertial>
-        <visual>
-        <origin xyz="0 0 0" rpy="0 0 0" />
-        <geometry>
-            <mesh filename="package://dual_piper_v2/meshes/dae/link7.dae" />
-        </geometry>
-        <material name="">
-            <color rgba="0.792156862745098 0.819607843137255 0.933333333333333 1" />
-        </material>
-        </visual>
-        <collision>
-        <origin xyz="0 0 0" rpy="0 0 0" />
-        <geometry>
-            <mesh filename="package://dual_piper_v2/meshes/dae/link7.dae" />
-        </geometry>
-        </collision>
-    </link>
-    <joint name="${namespace}/joint7" type="fixed">
-        <origin xyz="0 0 0.13503" rpy="1.5708 0 1.5708" />
-        <parent link="${namespace}/link6" />
-        <child link="${namespace}/link7" />
-        <axis xyz="0 0 -1" />
-        <limit lower="0" upper="0.05" effort="100" velocity="1" />
-    </joint>
-    <link name="${namespace}/link8">
-        <inertial>
-        <origin
-            xyz="0.000277816920932317 0.0467673824063769 -0.00921030054508036"
-            rpy="0 0 0" />
-        <mass value="0.0264822021416248" />
-        <inertia
-            ixx="9.99779119357223E-06"
-            ixy="-1.57542283433504E-07"
-            ixz="2.71367446701359E-08"
-            iyy="6.17952441557932E-06"
-            iyz="1.58939319453383E-06"
-            izz="1.4210192754512E-05" />
-        </inertial>
-        <visual>
-        <origin xyz="0 0 0" rpy="0 0 0" />
-        <geometry>
-            <mesh filename="package://dual_piper_v2/meshes/dae/link8.dae" />
-        </geometry>
-        <material name="">
-            <color rgba="0.792156862745098 0.819607843137255 0.933333333333333 1" />
-        </material>
-        </visual>
-        <collision>
-        <origin xyz="0 0 0" rpy="0 0 0" />
-        <geometry>
-            <mesh filename="package://dual_piper_v2/meshes/dae/link8.dae" />
-        </geometry>
-        </collision>
-    </link>
-    <joint name="${namespace}/joint8" type="fixed">
-        <origin xyz="0 0 0.13503" rpy="-1.5708 0 1.5708" />
-        <parent link="${namespace}/link6" />
-        <child link="${namespace}/link8" />
-        <axis xyz="0 0 1" />
-        <limit lower="-0.05" upper="0" effort="100" velocity="1" />
-    </joint> -->
 </xacro:macro>
 </robot>

File: ROS2/dual_piper_v2/urdf/piper_tenth.xacro (robot description, xacro)
@@ -29,7 +29,7 @@
         </inertial>
         <visual name="">
-            <origin xyz="0.057 0.0 -0.025" rpy="0.0 0.0 0.0"/>
+            <origin xyz="0.00 0.0 -0.15" rpy="0.0 0.0 -1.57"/>
             <geometry>
-                <mesh filename="package://dual_piper_v2/meshes/site.stl" />
+                <mesh filename="package://dual_piper_v2/meshes/site_v2.stl" />
             </geometry>
             <material name="">
@@ -45,6 +45,36 @@
         </collision>
     </link>
+    <!-- <link name="wall_link">
+        <inertial>
+            <origin xyz="0.0 0.0 0.0" rpy="0.0 0.0 0.0"/>
+            <mass value="0.0"/>
+            <inertia ixx="0.0" ixy="0.0" ixz="0.0" iyy="0.0" iyz="0.0" izz="0.0"/>
+        </inertial>
+        <visual name="">
+            <origin xyz="0.0 0.0 0.0" rpy="0.0 0.0 0.0"/>
+            <geometry>
+                <box size="0.01 5 5"/>
+            </geometry>
+            <material name="">
+                <color rgba="0.5 0.5 0.5 1.0"/>
+                <texture filename=""/>
+            </material>
+        </visual>
+        <collision>
+            <origin xyz="0.0 0.0 0.0" rpy="0.0 0.0 0.0"/>
+            <geometry>
+                <box size="0.01 5 5"/>
+            </geometry>
+        </collision>
+    </link>
+    <joint name="wall_joint" type="fixed">
+        <origin xyz="-1.25 0.0 0.0" rpy="0.0 0.0 0.0"/>
+        <parent link="arm_base_link"/>
+        <child link="wall_link"/>
+        <axis xyz="0.0 0.0 0.0"/>
+        <limit lower="0.0" upper="0.0" effort="0.0" velocity="0.0"/>
+    </joint> -->
     <joint name="piper_1_arm" type="fixed">
-        <origin xyz="0.63415 1.20559 0.0" rpy="0.0 0.0 0.0"/>
+        <origin xyz="0.45 1.29 0.03" rpy="0.0 0.0 1.57"/>
         <parent link="arm_base_link"/>
         <child link="piper_1/arm_base"/>
@@ -53,5 +83,5 @@
     </joint>
     <joint name="piper_2_arm" type="fixed">
-        <origin xyz="0.0 1.20559 0.0" rpy="0.0 0.0 0.0"/>
+        <origin xyz="-0.19 1.29 0.02" rpy="0.0 0.0 1.57"/>
         <parent link="arm_base_link"/>
         <child link="piper_2/arm_base"/>
@@ -60,5 +90,5 @@
     </joint>
     <joint name="piper_3_arm" type="fixed">
-        <origin xyz="-0.63415 1.20559 0.0" rpy="0.0 0.0 0.0"/>
+        <origin xyz="-0.83 1.29 0.09" rpy="0.0 0.0 1.57"/>
         <parent link="arm_base_link"/>
         <child link="piper_3/arm_base"/>
@@ -67,5 +97,5 @@
     </joint>
     <joint name="piper_4_arm" type="fixed">
-        <origin xyz="0.63415 0.72641 0.0" rpy="0.0 0.0 0.0"/>
+        <origin xyz="0.95 0.91 0.015" rpy="0.0 0.0 0.0"/>
         <parent link="arm_base_link"/>
         <child link="piper_4/arm_base"/>
@@ -74,5 +104,5 @@
     </joint>
     <joint name="piper_5_arm" type="fixed">
-        <origin xyz="0.63415 0.24341 0.0" rpy="0.0 0.0 0.0"/>
+        <origin xyz="0.95 0.25 0.025" rpy="0.0 0.0 0.0"/>
         <parent link="arm_base_link"/>
         <child link="piper_5/arm_base"/>
@@ -81,5 +111,5 @@
     </joint>
     <joint name="piper_6_arm" type="fixed">
-        <origin xyz="0.63415 -0.24341 0.0" rpy="0.0 0.0 0.0"/>
+        <origin xyz="0.95 -0.25 0.045" rpy="0.0 0.0 0.0"/>
         <parent link="arm_base_link"/>
         <child link="piper_6/arm_base"/>
@@ -88,5 +118,5 @@
     </joint>
     <joint name="piper_7_arm" type="fixed">
-        <origin xyz="0.63415 -0.72641 0.0" rpy="0.0 0.0 0.0"/>
+        <origin xyz="0.95 -0.91 0.015" rpy="0.0 0.0 0.0"/>
         <parent link="arm_base_link"/>
         <child link="piper_7/arm_base"/>
@@ -95,5 +125,5 @@
     </joint>
     <joint name="piper_8_arm" type="fixed">
-        <origin xyz="-0.63415 -1.20559 0.0" rpy="0.0 0.0 0.0"/>
+        <origin xyz="-0.83 -1.29 0.13" rpy="0.0 0.0 -1.57"/>
         <parent link="arm_base_link"/>
         <child link="piper_8/arm_base"/>
@@ -102,5 +132,5 @@
     </joint>
     <joint name="piper_9_arm" type="fixed">
-        <origin xyz="0.0 -1.20559  0.0" rpy="0.0 0.0 0.0"/>
+        <origin xyz="-0.19 -1.29  0.05" rpy="0.0 0.0 -1.57"/>
         <parent link="arm_base_link"/>
         <child link="piper_9/arm_base"/>
@@ -109,5 +139,5 @@
     </joint>
     <joint name="piper_10_arm" type="fixed">
-        <origin xyz="0.63415 -1.20559 0.0" rpy="0.0 0.0 0.0"/>
+        <origin xyz="0.45 -1.29 0.03" rpy="0.0 0.0 -1.57"/>
         <parent link="arm_base_link"/>
         <child link="piper_10/arm_base"/>
